Commit message: Before fixing IKP

File: autonomous_car/urdf/mobile_robot.urdf.xacro (robot description, xacro)
@@ -7,11 +7,11 @@
         <inertial>
             <origin xyz="0 0 0" rpy="0.0 0.0 0.0"/>
-            <mass value="30.0"/>
-            <inertia ixx="0.0" ixy="0.0" ixz="0.0" iyy="0.0" iyz="0.0" izz="0.0"/>
+            <mass value="45.0"/>
+            <inertia ixx="0.1" ixy="0.0" ixz="0.0" iyy="0.09101576355" iyz="0.0" izz="0.11243841101"/>
         </inertial>
         <visual>
-            <origin xyz="-1 0.5 -0.025" rpy="1.5708 0.0 0.0"/>
+            <origin xyz="0.0 -0.0 0.05" rpy="0.0 0.0 0.0"/>
             <geometry>
-                <mesh filename="package://autonomous_car/meshes/badane.STL" scale="0.001 0.001 0.001"/>
+                <box size="0.8 0.44 0.09"/>
             </geometry>
             <material name="">
@@ -20,7 +20,7 @@
         </visual>
         <collision>
-            <origin xyz="-1 0.5 -0.025" rpy="1.5708 0.0 0.0"/>
+            <origin xyz="0.0 -0.0 0.05" rpy="0.0 0.0 0.0"/>
             <geometry>
-                <mesh filename="package://autonomous_car/meshes/badane.STL" scale="0.001 0.001 0.001"/>
+                <box size="0.8 0.44 0.09"/>
             </geometry>
         </collision>
@@ -47,5 +47,5 @@
         </visual>
         <inertial>
-          <mass value="1" />
+          <mass value="0" />
           <origin xyz="0 0 0" rpy="0 0 0"/>
           <inertia ixx="0" ixy="0" ixz="0" iyy="0" iyz="0" izz="0" />
@@ -53,6 +53,6 @@
     </link>
     <joint name="camera_sensor_joint" type="fixed">
-        <origin xyz="0.0 0.0 0.5" rpy="0.0 0.0 0.0"/>
-        <parent link="front_steering"/>
+        <origin xyz="0.35 0.0 0.125" rpy="0.0 0.0 0.0"/>
+        <parent link="car_body"/>
         <child link="camera_sensor_link"/>
         <axis xyz="0.0 0.0 0.0"/>
@@ -62,6 +62,6 @@
         <inertial>
             <origin xyz="0.0 0.0 0.0" rpy="0.0 0.0 0.0"/>
-            <mass value="1.0"/>
-            <inertia ixx="0.0" ixy="0.0" ixz="0.0" iyy="0.0" iyz="0.0" izz="0.0"/>
+            <mass value="0.0"/>
+            <inertia ixx="0.01" ixy="0.0" ixz="0.0" iyy="0.01" iyz="0.0" izz="0.01"/>
         </inertial>
         <visual name="">
@@ -83,73 +83,9 @@
     </link>
     <joint name="IMU_sensor_joint" type="fixed">
-        <origin xyz="0.0 0.0 0.5" rpy="0.0 0.0 0.0"/>
+        <origin xyz="0.0 0.0 0.125" rpy="0.0 0.0 0.0"/>
         <parent link="car_body"/>
         <child link="IMU_sensor_link"/>
         <axis xyz="0.0 0.0 0.0"/>
         <limit lower="0.0" upper="0.0" effort="0.0" velocity="0.0"/>
-    </joint>
-    <!-- Include Contact sensors URDFs -->
-    <!-- <xacro:include filename="front_sensors.urdf.xacro"/>
-    <xacro:include filename="rear_sensors.urdf.xacro"/>
-    <xacro:include filename="side_sensors.urdf.xacro"/>
-    <xacro:include filename="corner_sensors.urdf.xacro"/> -->
-    <!-- Steering of the car -->
-    <!-- Back Steering -->
-    <link name="back_steering">
-        <inertial>
-            <origin xyz="0 0 0"  rpy="0.0 0.0 0.0"/>
-            <mass value="1.0"/>
-            <inertia ixx="0.0" ixy="0.0" ixz="0.0" iyy="0.0" iyz="0.0" izz="0.0"/>
-        </inertial>
-        <visual>
-            <origin xyz="0 0.0 0.125" rpy="1.5708 0.0 0.0"/>
-            <geometry>
-                <cylinder radius="0.05" length="1.5"/>
-            </geometry>
-            <material name="">
-                <color rgba="1.0 0.0 0.0 1.0"/>
-            </material>
-        </visual>
-        <collision>
-            <origin xyz="0 0.0 0.125" rpy="1.5708 0.0 0.0"/>
-            <geometry>
-                <cylinder radius="0.05" length="1.5"/>
-            </geometry>
-        </collision>
-    </link>
-    <joint name="back_steering_joint" type="fixed">
-        <origin xyz="-0.85 0.0 0.0" rpy="0.0 0.0 0.0"/>
-        <parent link="car_body"/>
-        <child link="back_steering"/>
-        <axis xyz="0.0 0.0 0.0"/>
-    </joint>
-    <!-- Front steering -->
-    <link name="front_steering">
-        <inertial>
-            <origin xyz="0 0 0"  rpy="0.0 0.0 0.0"/>
-            <mass value="1.0"/>
-            <inertia ixx="0.0" ixy="0.0" ixz="0.0" iyy="0.0" iyz="0.0" izz="0.0"/>
-        </inertial>
-        <visual>
-            <origin xyz="0 0.0 0.125" rpy="1.5708 0.0 0.0"/>
-            <geometry>
-                <cylinder radius="0.05" length="1.5"/>
-            </geometry>
-            <material name="">
-                <color rgba="1.0 0.0 0.0 1.0"/>
-            </material>
-        </visual>
-        <collision>
-            <origin xyz="0 0.0 0.125" rpy="1.5708 0.0 0.0"/>
-            <geometry>
-                <cylinder radius="0.05" length="1.5"/>
-            </geometry>
-        </collision>
-    </link>
-    <joint name="front_steering_joint" type="fixed">
-        <origin xyz="0.85 0.0 0.0" rpy="0.0 0.0 0.0"/>
-        <parent link="car_body"/>
-        <child link="front_steering"/>
-        <axis xyz="0.0 0.0 0.0"/>
     </joint>
     <!-- Wheels -->
@@ -158,22 +94,22 @@
         <inertial>
             <origin xyz="0.0 0.0 0.0" rpy="0.0 0.0 0.0"/>
-            <mass value="1.431"/>
-            <inertia ixx="0.0" ixy="0.0" ixz="0.0" iyy="0.0" iyz="0.0" izz="0.0"/>
+            <mass value="0.8"/>
+            <inertia ixx="0.01" ixy="0.0" ixz="0.0" iyy="0.01" iyz="0.0" izz="0.01"/>
         </inertial>
         <visual>
-            <origin xyz="-0.25 0.1 -0.25" rpy="1.5707 0.0 0.0"/>
+            <origin xyz="0.0 -0.0 0.0" rpy="1.5708 0.0 0.0"/>
             <geometry>
-                <mesh filename="package://autonomous_car/meshes/charkh.STL" scale="0.001 0.001 0.001"/>
+                <cylinder radius="0.0975" length="0.06"/>
             </geometry>
         </visual>
         <collision>
-            <origin xyz="-0.25 0.1 -0.25" rpy="1.5707 0.0 0.0"/>
+            <origin xyz="0.0 -0.0 0.0" rpy="1.5708 0.0 0.0"/>
             <geometry>
-                <mesh filename="package://autonomous_car/meshes/charkh.STL" scale="0.001 0.001 0.001"/>
+                <cylinder radius="0.0975" length="0.06"/>
             </geometry>
         </collision>
     </link>
     <joint name="right_wheel_joint" type="continuous">
-        <origin xyz="0.85 0.6 0.125" rpy="0.0 0.0 0.0"/>
+        <origin xyz="0.35 0.25 0.03" rpy="0.0 0.0 0.0"/>
         <parent link="car_body"/>
         <child link="right_wheel"/>
@@ -184,22 +120,22 @@
         <inertial>
             <origin xyz="0.0 0.0 0.0" rpy="0.0 0.0 0.0"/>
-            <mass value="1.431"/>
-            <inertia ixx="0.0" ixy="0.0" ixz="0.0" iyy="0.0" iyz="0.0" izz="0.0"/>
+            <mass value="0.8"/>
+            <inertia ixx="0.01" ixy="0.0" ixz="0.0" iyy="0.01" iyz="0.0" izz="0.01"/>
         </inertial>
         <visual>
-            <origin xyz="-0.25 0.1 -0.25"  rpy="1.5707 0.0 0.0"/>
+            <origin xyz="0.0 -0.0 0.0" rpy="1.5708 0.0 0.0"/>
             <geometry>
-                <mesh filename="package://autonomous_car/meshes/charkh.STL" scale="0.001 0.001 0.001"/>
+                <cylinder radius="0.0975" length="0.06"/>
             </geometry>
         </visual>
         <collision>
-            <origin xyz="-0.25 0.1 -0.25" rpy="1.5707 0.0 0.0"/>
+            <origin xyz="0.0 -0.0 0.0" rpy="1.5708 0.0 0.0"/>
             <geometry>
-                <mesh filename="package://autonomous_car/meshes/charkh.STL" scale="0.001 0.001 0.001"/>
+                <cylinder radius="0.0975" length="0.06"/>
             </geometry>
         </collision>
     </link>
     <joint name="left_wheel_joint" type="continuous">
-        <origin xyz="0.85 -0.6 0.125" rpy="0.0 0.0 0.0"/>
+        <origin xyz="0.35 -0.25 0.03" rpy="0.0 0.0 0.0"/>
         <parent link="car_body"/>
         <child link="left_wheel"/>
@@ -209,22 +145,22 @@
         <inertial>
             <origin xyz="0.0 0.0 0.0" rpy="0.0 0.0 0.0"/>
-            <mass value="1.431"/>
-            <inertia ixx="0.0" ixy="0.0" ixz="0.0" iyy="0.0" iyz="0.0" izz="0.0"/>
+            <mass value="0.8"/>
+            <inertia ixx="0.01" ixy="0.0" ixz="0.0" iyy="0.01" iyz="0.0" izz="0.01"/>
         </inertial>
         <visual>
-            <origin xyz="-0.25 0.10 -0.25" rpy="1.5707 0.0 0.0"/>
+            <origin xyz="0.0 -0.0 0.0" rpy="1.5708 0.0 0.0"/>
             <geometry>
-                <mesh filename="package://autonomous_car/meshes/charkh.STL" scale="0.001 0.001 0.001"/>
+                <cylinder radius="0.0975" length="0.06"/>
             </geometry>
         </visual>
         <collision>
-            <origin xyz="-0.25 0.10 -0.25" rpy="1.5707 0.0 0.0"/>
+            <origin xyz="0.0 -0.0 0.0" rpy="1.5708 0.0 0.0"/>
             <geometry>
-                <mesh filename="package://autonomous_car/meshes/charkh.STL" scale="0.001 0.001 0.001"/>
+                <cylinder radius="0.0975" length="0.06"/>
             </geometry>
         </collision>
     </link>
     <joint name="left_back_wheel_joint" type="continuous">
-        <origin xyz="-0.85 -0.6 0.125" rpy="0.0 0.0 0.0"/>
+        <origin xyz="-0.3 -0.25 0.03" rpy="0.0 0.0 0.0"/>
         <parent link="car_body"/>
         <child link="left_back_wheel"/>
@@ -234,22 +170,22 @@
         <inertial>
             <origin xyz="0.0 0.0 0.0" rpy="0.0 0.0 0.0"/>
-            <mass value="1.431"/>
-            <inertia ixx="0.0" ixy="0.0" ixz="0.0" iyy="0.0" iyz="0.0" izz="0.0"/>
+            <mass value="0.8"/>
+            <inertia ixx="0.01" ixy="0.0" ixz="0.0" iyy="0.01" iyz="0.0" izz="0.01"/>
         </inertial>
         <visual>
-            <origin xyz="-0.25 0.10 -0.25" rpy="1.5707 0.0 0.0"/>
+            <origin xyz="0.0 -0.0 0.0" rpy="1.5708 0.0 0.0"/>
             <geometry>
-                <mesh filename="package://autonomous_car/meshes/charkh.STL" scale="0.001 0.001 0.001"/>
+                <cylinder radius="0.0975" length="0.06"/>
             </geometry>
         </visual>
         <collision>
-            <origin xyz="-0.25 0.10 -0.25" rpy="1.5707 0.0 0.0"/>
+            <origin xyz="0.0 -0.0 0.0" rpy="1.5708 0.0 0.0"/>
             <geometry>
-                <mesh filename="package://autonomous_car/meshes/charkh.STL" scale="0.001 0.001 0.001"/>
+                <cylinder radius="0.0975" length="0.06"/>
             </geometry>
         </collision>
     </link>
     <joint name="right_back_wheel_joint" type="continuous">
-        <origin xyz="-0.85 0.6 0.125" rpy="0.0 0.0 0.0"/>
+        <origin xyz="-0.3 0.25 0.03" rpy="0.0 0.0 0.0"/>
         <parent link="car_body"/>
         <child link="right_back_wheel"/>

File: autonomous_car/urdf/simulation_gazebo.xacro (robot description, xacro)
@@ -1,58 +1,58 @@
 <?xml version="1.0"?>
 <robot xmlns:xacro="http://www.ros.org/wiki/xacro" name="mobile_robot_description">
-    <transmission name="right_wheel_transmition">
-        <type>transmission_interface/SimpleTransmission</type>
-        <joint name="right_wheel_joint">
-            <hardwareInterface>hardware_interface/VelocityJointInterface</hardwareInterface>
-        </joint>
-        <actuator name="right_wheel_motor">
-            <mechanicalReduction>1.0</mechanicalReduction>
-            <hardwareInterface>hardware_interface/VelocityJointInterface</hardwareInterface>
-        </actuator>
-    </transmission>
-    <transmission name="left_wheel_transmition">
-        <type>transmission_interface/SimpleTransmission</type>
-        <joint name="left_wheel_joint">
-            <hardwareInterface>hardware_interface/VelocityJointInterface</hardwareInterface>
-        </joint>
-        <actuator name="left_wheel_motor">
-            <mechanicalReduction>1.0</mechanicalReduction>
-            <hardwareInterface>hardware_interface/VelocityJointInterface</hardwareInterface>
-        </actuator>
-    </transmission>
-    <gazebo refrence="right_wheel">
-        <mu1>0.4</mu1>
-        <mu2>0.4</mu2>
+  <transmission name="right_wheel_transmition">
+    <type>transmission_interface/SimpleTransmission</type>
+    <joint name="right_wheel_joint">
+        <hardwareInterface>hardware_interface/VelocityJointInterface</hardwareInterface>
+    </joint>
+    <actuator name="right_wheel_motor">
+        <mechanicalReduction>1.0</mechanicalReduction>
+        <hardwareInterface>hardware_interface/VelocityJointInterface</hardwareInterface>
+    </actuator>
+</transmission>
+<transmission name="left_wheel_transmition">
+    <type>transmission_interface/SimpleTransmission</type>
+    <joint name="left_wheel_joint">
+        <hardwareInterface>hardware_interface/VelocityJointInterface</hardwareInterface>
+    </joint>
+    <actuator name="left_wheel_motor">
+        <mechanicalReduction>1.0</mechanicalReduction>
+        <hardwareInterface>hardware_interface/VelocityJointInterface</hardwareInterface>
+    </actuator>
+</transmission>
+    <gazebo reference="right_wheel">
+        <mu1>0.6</mu1>
+        <mu2>0.6</mu2>
         <kp>1000000</kp>
         <kd>1000</kd>
         <minDepth>0.001</minDepth>
-        <maxVel>0.1</maxVel>
+        <maxVel>3</maxVel>
         <fdir>1 0 0</fdir>
     </gazebo>
-    <gazebo refrence="left_wheel">
-        <mu1>0.4</mu1>
-        <mu2>0.4</mu2>
+    <gazebo reference="left_wheel">
+        <mu1>0.6</mu1>
+        <mu2>0.6</mu2>
         <kp>1000000</kp>
         <kd>1000</kd>
         <minDepth>0.001</minDepth>
-        <maxVel>0.1</maxVel>
+        <maxVel>3</maxVel>
         <fdir>1 0 0</fdir>
     </gazebo>
-    <gazebo refrence="left_back_wheel">
-        <mu1>0.4</mu1>
-        <mu2>0.4</mu2>
+    <gazebo reference="left_back_wheel">
+        <mu1>0.6</mu1>
+        <mu2>0.6</mu2>
         <kp>1000000</kp>
         <kd>1000</kd>
         <minDepth>0.001</minDepth>
-        <maxVel>0.1</maxVel>
+        <maxVel>3</maxVel>
         <fdir>1 0 0</fdir>
     </gazebo>
-    <gazebo refrence="right_back_wheel">
-        <mu1>0.4</mu1>
-        <mu2>0.4</mu2>
+    <gazebo reference="right_back_wheel">
+        <mu1>0.6</mu1>
+        <mu2>0.6</mu2>
         <kp>1000000</kp>
         <kd>1000</kd>
         <minDepth>0.001</minDepth>
-        <maxVel>0.1</maxVel>
+        <maxVel>3</maxVel>
         <fdir>1 0 0</fdir>
     </gazebo>
@@ -91,7 +91,7 @@
           <distortionT1>0.00000001</distortionT1>
           <distortionT2>0.00000001</distortionT2>
-          <Cx>400</Cx> <!-- Principal point x in pixels (width/2) -->
-          <Cy>300</Cy> <!-- Principal point y in pixels (height/2) -->
-          <focalLength>692.818364</focalLength> <!-- Updated focal length -->
+          <Cx>400</Cx>
+          <Cy>300</Cy>
+          <focalLength>692.818364</focalLength>
           <hackBaseline>0</hackBaseline>
         </plugin>

Commit message: Fixing IKP

File: autonomous_car/urdf/mobile_robot.urdf.xacro (robot description, xacro)
@@ -8,5 +8,5 @@
             <origin xyz="0 0 0" rpy="0.0 0.0 0.0"/>
             <mass value="45.0"/>
-            <inertia ixx="0.1" ixy="0.0" ixz="0.0" iyy="0.09101576355" iyz="0.0" izz="0.11243841101"/>
+            <inertia ixx="0.50425" ixy="0.0" ixz="0.0" iyy="1.6202500000000004" iyz="0.0" izz="2.0840000000000005" />
         </inertial>
         <visual>
@@ -63,5 +63,5 @@
             <origin xyz="0.0 0.0 0.0" rpy="0.0 0.0 0.0"/>
             <mass value="0.0"/>
-            <inertia ixx="0.01" ixy="0.0" ixz="0.0" iyy="0.01" iyz="0.0" izz="0.01"/>
+            <inertia ixx="0.002" ixy="0.0" ixz="0.0" iyy="0.002" iyz="0.0" izz="0.0038"/>
         </inertial>
         <visual name="">
@@ -95,5 +95,5 @@
             <origin xyz="0.0 0.0 0.0" rpy="0.0 0.0 0.0"/>
             <mass value="0.8"/>
-            <inertia ixx="0.01" ixy="0.0" ixz="0.0" iyy="0.01" iyz="0.0" izz="0.01"/>
+            <inertia ixx="0.002" ixy="0.0" ixz="0.0" iyy="0.002" iyz="0.0" izz="0.0038"/>
         </inertial>
         <visual>
@@ -121,5 +121,5 @@
             <origin xyz="0.0 0.0 0.0" rpy="0.0 0.0 0.0"/>
             <mass value="0.8"/>
-            <inertia ixx="0.01" ixy="0.0" ixz="0.0" iyy="0.01" iyz="0.0" izz="0.01"/>
+            <inertia ixx="0.002" ixy="0.0" ixz="0.0" iyy="0.002" iyz="0.0" izz="0.0038"/>
         </inertial>
         <visual>
@@ -146,5 +146,5 @@
             <origin xyz="0.0 0.0 0.0" rpy="0.0 0.0 0.0"/>
             <mass value="0.8"/>
-            <inertia ixx="0.01" ixy="0.0" ixz="0.0" iyy="0.01" iyz="0.0" izz="0.01"/>
+            <inertia ixx="0.002" ixy="0.0" ixz="0.0" iyy="0.002" iyz="0.0" izz="0.0038"/>
         </inertial>
         <visual>
@@ -171,5 +171,5 @@
             <origin xyz="0.0 0.0 0.0" rpy="0.0 0.0 0.0"/>
             <mass value="0.8"/>
-            <inertia ixx="0.01" ixy="0.0" ixz="0.0" iyy="0.01" iyz="0.0" izz="0.01"/>
+            <inertia ixx="0.002" ixy="0.0" ixz="0.0" iyy="0.002" iyz="0.0" izz="0.0038"/>
         </inertial>
         <visual>

File: autonomous_car/urdf/simulation_gazebo.xacro (robot description, xacro)
@@ -22,6 +22,6 @@
 </transmission>
     <gazebo reference="right_wheel">
-        <mu1>0.6</mu1>
-        <mu2>0.6</mu2>
+        <mu1>0.8</mu1>
+        <mu2>0.8</mu2>
         <kp>1000000</kp>
         <kd>1000</kd>
@@ -31,6 +31,6 @@
     </gazebo>
     <gazebo reference="left_wheel">
-        <mu1>0.6</mu1>
-        <mu2>0.6</mu2>
+        <mu1>0.8</mu1>
+        <mu2>0.8</mu2>
         <kp>1000000</kp>
         <kd>1000</kd>
@@ -40,6 +40,6 @@
     </gazebo>
     <gazebo reference="left_back_wheel">
-        <mu1>0.6</mu1>
-        <mu2>0.6</mu2>
+        <mu1>0.8</mu1>
+        <mu2>0.8</mu2>
         <kp>1000000</kp>
         <kd>1000</kd>
@@ -49,6 +49,6 @@
     </gazebo>
     <gazebo reference="right_back_wheel">
-        <mu1>0.6</mu1>
-        <mu2>0.6</mu2>
+        <mu1>0.8</mu1>
+        <mu2>0.8</mu2>
         <kp>1000000</kp>
         <kd>1000</kd>

Commit message: Added APF-RL method

File: autonomous_car/urdf/mobile_robot.urdf.xacro (robot description, xacro)
@@ -7,6 +7,8 @@
         <inertial>
             <origin xyz="0 0 0" rpy="0.0 0.0 0.0"/>
-            <mass value="45.0"/>
-            <inertia ixx="0.50425" ixy="0.0" ixz="0.0" iyy="1.6202500000000004" iyz="0.0" izz="2.0840000000000005" />
+            <mass value="15.0"/>
+            <inertia ixx="0.25" ixy="0.0" ixz="0.0"
+             iyy="0.81" iyz="0.0"
+             izz="1" />
         </inertial>
         <visual>
@@ -87,5 +89,4 @@
         <child link="IMU_sensor_link"/>
         <axis xyz="0.0 0.0 0.0"/>
-        <limit lower="0.0" upper="0.0" effort="0.0" velocity="0.0"/>
     </joint>
     <!-- Wheels -->
@@ -93,5 +94,5 @@
     <link name="right_wheel">
         <inertial>
-            <origin xyz="0.0 0.0 0.0" rpy="0.0 0.0 0.0"/>
+            <origin xyz="0.0 0.0 0.0" rpy="1.5708 0.0 0.0"/>
             <mass value="0.8"/>
             <inertia ixx="0.002" ixy="0.0" ixz="0.0" iyy="0.002" iyz="0.0" izz="0.0038"/>
@@ -119,5 +120,5 @@
     <link name="left_wheel">
         <inertial>
-            <origin xyz="0.0 0.0 0.0" rpy="0.0 0.0 0.0"/>
+            <origin xyz="0.0 0.0 0.0" rpy="1.5708 0.0 0.0"/>
             <mass value="0.8"/>
             <inertia ixx="0.002" ixy="0.0" ixz="0.0" iyy="0.002" iyz="0.0" izz="0.0038"/>
@@ -144,5 +145,5 @@
     <link name="left_back_wheel">
         <inertial>
-            <origin xyz="0.0 0.0 0.0" rpy="0.0 0.0 0.0"/>
+            <origin xyz="0.0 0.0 0.0" rpy="1.5708 0.0 0.0"/>
             <mass value="0.8"/>
             <inertia ixx="0.002" ixy="0.0" ixz="0.0" iyy="0.002" iyz="0.0" izz="0.0038"/>
@@ -162,5 +163,5 @@
     </link>
     <joint name="left_back_wheel_joint" type="continuous">
-        <origin xyz="-0.3 -0.25 0.03" rpy="0.0 0.0 0.0"/>
+        <origin xyz="-0.35 -0.25 0.03" rpy="0.0 0.0 0.0"/>
         <parent link="car_body"/>
         <child link="left_back_wheel"/>
@@ -169,5 +170,5 @@
     <link name="right_back_wheel">
         <inertial>
-            <origin xyz="0.0 0.0 0.0" rpy="0.0 0.0 0.0"/>
+            <origin xyz="0.0 0.0 0.0" rpy="1.5708 0.0 0.0"/>
             <mass value="0.8"/>
             <inertia ixx="0.002" ixy="0.0" ixz="0.0" iyy="0.002" iyz="0.0" izz="0.0038"/>
@@ -187,5 +188,5 @@
     </link>
     <joint name="right_back_wheel_joint" type="continuous">
-        <origin xyz="-0.3 0.25 0.03" rpy="0.0 0.0 0.0"/>
+        <origin xyz="-0.35 0.25 0.03" rpy="0.0 0.0 0.0"/>
         <parent link="car_body"/>
         <child link="right_back_wheel"/>

File: autonomous_car/urdf/simulation_gazebo.xacro (robot description, xacro)
@@ -1,5 +1,5 @@
 <?xml version="1.0"?>
 <robot xmlns:xacro="http://www.ros.org/wiki/xacro" name="mobile_robot_description">
-  <transmission name="right_wheel_transmition">
+  <!-- <transmission name="right_wheel_transmition">
     <type>transmission_interface/SimpleTransmission</type>
     <joint name="right_wheel_joint">
@@ -20,10 +20,30 @@
         <hardwareInterface>hardware_interface/VelocityJointInterface</hardwareInterface>
     </actuator>
-</transmission>
+</transmission> -->
+    <gazebo>
+      <plugin name="skid_steering_controller" filename="libgazebo_ros_skid_steer_drive.so">
+        <updateRate>100.0</updateRate>
+        <robotNamespace>/</robotNamespace>
+        <leftFrontJoint>right_wheel_joint</leftFrontJoint>
+        <rightFrontJoint>left_wheel_joint</rightFrontJoint>
+        <leftRearJoint>right_back_wheel_joint</leftRearJoint>
+        <rightRearJoint>left_back_wheel_joint</rightRearJoint>
+        <wheelSeparation>0.5</wheelSeparation>
+        <wheelDiameter>0.195</wheelDiameter>
+        <robotBaseFrame>base_link</robotBaseFrame>
+        <torque>500</torque>
+        <topicName>cmd_vel</topicName>
+        <broadcastTF>false</broadcastTF>
+      </plugin>
+    </gazebo>
+    <gazebo reference="car_body">
+      <mu1>0.2</mu1>
+      <mu2>1</mu2>
+    </gazebo>
     <gazebo reference="right_wheel">
-        <mu1>0.8</mu1>
-        <mu2>0.8</mu2>
+        <mu1>0.2</mu1>
+        <mu2>1</mu2>
         <kp>1000000</kp>
-        <kd>1000</kd>
+        <kd>100</kd>
         <minDepth>0.001</minDepth>
         <maxVel>3</maxVel>
@@ -31,8 +51,8 @@
     </gazebo>
     <gazebo reference="left_wheel">
-        <mu1>0.8</mu1>
-        <mu2>0.8</mu2>
+        <mu1>0.2</mu1>
+        <mu2>1</mu2>
         <kp>1000000</kp>
-        <kd>1000</kd>
+        <kd>100</kd>
         <minDepth>0.001</minDepth>
         <maxVel>3</maxVel>
@@ -40,8 +60,8 @@
     </gazebo>
     <gazebo reference="left_back_wheel">
-        <mu1>0.8</mu1>
-        <mu2>0.8</mu2>
+        <mu1>0.2</mu1>
+        <mu2>1</mu2>
         <kp>1000000</kp>
-        <kd>1000</kd>
+        <kd>100</kd>
         <minDepth>0.001</minDepth>
         <maxVel>3</maxVel>
@@ -49,8 +69,8 @@
     </gazebo>
     <gazebo reference="right_back_wheel">
-        <mu1>0.8</mu1>
-        <mu2>0.8</mu2>
+        <mu1>0.2</mu1>
+        <mu2>1</mu2>
         <kp>1000000</kp>
-        <kd>1000</kd>
+        <kd>100</kd>
         <minDepth>0.001</minDepth>
         <maxVel>3</maxVel>
@@ -74,5 +94,5 @@
         </camera>
         <plugin name="camera_controller" filename="libgazebo_ros_openni_kinect.so">
-          <baseline>0.2</baseline>
+          <baseline>0.1</baseline>
           <alwaysOn>true</alwaysOn>
           <updateRate>1.0</updateRate>
