Commit message: Remove Unnecessary files

File: autonomous_car/urdf/mobile_robot.urdf.xacro (robot description, xacro)
@@ -13,7 +13,7 @@
         </inertial>
         <visual>
-            <origin xyz="0.0 -0.0 0.05" rpy="0.0 0.0 0.0"/>
+            <origin xyz="0.5 -0.223 0.2" rpy="-1.5708 0.0 1.5708"/>
             <geometry>
-                <box size="0.8 0.44 0.09"/>
+                <mesh filename="package://autonomous_car/meshes/chasis.STL" scale="0.001 0.001 0.001"/>
             </geometry>
             <material name="">
@@ -22,7 +22,7 @@
         </visual>
         <collision>
-            <origin xyz="0.0 -0.0 0.05" rpy="0.0 0.0 0.0"/>
+            <origin xyz="0.5 -0.223 0.2" rpy="-1.5708 0.0 1.5708"/>
             <geometry>
-                <box size="0.8 0.44 0.09"/>
+                <mesh filename="package://autonomous_car/meshes/chasis.STL" scale="0.001 0.001 0.001"/>
             </geometry>
         </collision>
@@ -55,5 +55,5 @@
     </link>
     <joint name="camera_sensor_joint" type="fixed">
-        <origin xyz="0.35 0.0 0.125" rpy="0.0 0.0 0.0"/>
+        <origin xyz="0.35 0.0 0.225" rpy="0.0 0.0 0.0"/>
         <parent link="car_body"/>
         <child link="camera_sensor_link"/>
@@ -99,18 +99,18 @@
         </inertial>
         <visual>
-            <origin xyz="0.0 -0.0 0.0" rpy="1.5708 0.0 0.0"/>
+            <origin xyz="-0.0975 -0.03 -0.0975" rpy="1.5708 0.0 1.5708"/>
             <geometry>
-                <cylinder radius="0.0975" length="0.06"/>
+                <mesh filename="package://autonomous_car/meshes/wheel.STL" scale="0.001 0.001 0.001"/>
             </geometry>
         </visual>
         <collision>
-            <origin xyz="0.0 -0.0 0.0" rpy="1.5708 0.0 0.0"/>
+            <origin xyz="-0.0975 -0.03 -0.0975" rpy="1.5708 0.0 1.5708"/>
             <geometry>
-                <cylinder radius="0.0975" length="0.06"/>
+                <mesh filename="package://autonomous_car/meshes/wheel.STL" scale="0.001 0.001 0.001"/>
             </geometry>
         </collision>
     </link>
     <joint name="right_wheel_joint" type="continuous">
-        <origin xyz="0.35 0.25 0.03" rpy="0.0 0.0 0.0"/>
+        <origin xyz="0.35 0.26 0.03" rpy="0.0 0.0 0.0"/>
         <parent link="car_body"/>
         <child link="right_wheel"/>
@@ -125,13 +125,13 @@
         </inertial>
         <visual>
-            <origin xyz="0.0 -0.0 0.0" rpy="1.5708 0.0 0.0"/>
+            <origin xyz="0.0975 0.03 -0.0975" rpy="1.5708 0.0 -1.5708"/>
             <geometry>
-                <cylinder radius="0.0975" length="0.06"/>
+                <mesh filename="package://autonomous_car/meshes/wheel.STL" scale="0.001 0.001 0.001"/>
             </geometry>
         </visual>
         <collision>
-            <origin xyz="0.0 -0.0 0.0" rpy="1.5708 0.0 0.0"/>
+            <origin xyz="0.0975 0.03 -0.0975" rpy="1.5708 0.0 -1.5708"/>
             <geometry>
-                <cylinder radius="0.0975" length="0.06"/>
+                <mesh filename="package://autonomous_car/meshes/wheel.STL" scale="0.001 0.001 0.001"/>
             </geometry>
         </collision>
@@ -150,18 +150,18 @@
         </inertial>
         <visual>
-            <origin xyz="0.0 -0.0 0.0" rpy="1.5708 0.0 0.0"/>
+            <origin xyz="0.0975 0.03 -0.0975" rpy="1.5708 0.0 -1.5708"/>
             <geometry>
-                <cylinder radius="0.0975" length="0.06"/>
+                <mesh filename="package://autonomous_car/meshes/wheel.STL" scale="0.001 0.001 0.001"/>
             </geometry>
         </visual>
         <collision>
-            <origin xyz="0.0 -0.0 0.0" rpy="1.5708 0.0 0.0"/>
+            <origin xyz="0.0975 0.03 -0.0975" rpy="1.5708 0.0 -1.5708"/>
             <geometry>
-                <cylinder radius="0.0975" length="0.06"/>
+                <mesh filename="package://autonomous_car/meshes/wheel.STL" scale="0.001 0.001 0.001"/>
             </geometry>
         </collision>
     </link>
     <joint name="left_back_wheel_joint" type="continuous">
-        <origin xyz="-0.35 -0.25 0.03" rpy="0.0 0.0 0.0"/>
+        <origin xyz="-0.3 -0.25 0.03" rpy="0.0 0.0 0.0"/>
         <parent link="car_body"/>
         <child link="left_back_wheel"/>
@@ -175,18 +175,18 @@
         </inertial>
         <visual>
-            <origin xyz="0.0 -0.0 0.0" rpy="1.5708 0.0 0.0"/>
+            <origin xyz="-0.0975 -0.03 -0.0975" rpy="1.5708 0.0 1.5708"/>
             <geometry>
-                <cylinder radius="0.0975" length="0.06"/>
+                <mesh filename="package://autonomous_car/meshes/wheel.STL" scale="0.001 0.001 0.001"/>
             </geometry>
         </visual>
         <collision>
-            <origin xyz="0.0 -0.0 0.0" rpy="1.5708 0.0 0.0"/>
+            <origin xyz="-0.0975 -0.03 -0.0975" rpy="1.5708 0.0 1.5708"/>
             <geometry>
-                <cylinder radius="0.0975" length="0.06"/>
+                <mesh filename="package://autonomous_car/meshes/wheel.STL" scale="0.001 0.001 0.001"/>
             </geometry>
         </collision>
     </link>
     <joint name="right_back_wheel_joint" type="continuous">
-        <origin xyz="-0.35 0.25 0.03" rpy="0.0 0.0 0.0"/>
+        <origin xyz="-0.30 0.26 0.03" rpy="0.0 0.0 0.0"/>
         <parent link="car_body"/>
         <child link="right_back_wheel"/>

File: autonomous_car/urdf/simulation_gazebo.xacro (robot description, xacro)
@@ -39,9 +39,9 @@
     <gazebo reference="car_body">
       <mu1>0.2</mu1>
-      <mu2>1</mu2>
+      <mu2>0.5</mu2>
     </gazebo>
     <gazebo reference="right_wheel">
         <mu1>0.2</mu1>
-        <mu2>1</mu2>
+        <mu2>0.5</mu2>
         <kp>1000000</kp>
         <kd>100</kd>
@@ -52,5 +52,5 @@
     <gazebo reference="left_wheel">
         <mu1>0.2</mu1>
-        <mu2>1</mu2>
+        <mu2>0.5</mu2>
         <kp>1000000</kp>
         <kd>100</kd>
@@ -61,5 +61,5 @@
     <gazebo reference="left_back_wheel">
         <mu1>0.2</mu1>
-        <mu2>1</mu2>
+        <mu2>0.5</mu2>
         <kp>1000000</kp>
         <kd>100</kd>
@@ -70,5 +70,5 @@
     <gazebo reference="right_back_wheel">
         <mu1>0.2</mu1>
-        <mu2>1</mu2>
+        <mu2>0.5</mu2>
         <kp>1000000</kp>
         <kd>100</kd>
